File: pcb/_autosave-crime_hat.kicad_sch (KiCad schematic)
At the start: 7 parts, among them J1 Conn_01x02_Male, Q1 2N2222, Q2 FQP27P06

Commit message: layout
Parts:
- D2: footprint (none) -> LED_THT:Chanzon_LED
Changed lines of the file:
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@@
       (effects (font (size 1.27 1.27)) (justify right))
     )
-    (property "Footprint" "" (id 2) (at 158.75 102.87 0)
+    (property "Footprint" "LED_THT:Chanzon_LED" (id 2) (at 158.75 102.87 0)
       (effects (font (size 1.27 1.27)) hide)
     )
@@
     )
     (path "/82b93f1d-8bb7-41d3-935d-a480541108f5"
-      (reference "D2") (unit 1) (value "LED") (footprint "")
+      (reference "D2") (unit 1) (value "LED") (footprint "LED_THT:Chanzon_LED")
     )
     (path "/2969ecd2-ca66-45d3-8f4b-c7ccf3a45bef"
